Commit message: fixed urdf file

File: install/robot_description/share/robot_description/urdf/robot.urdf.xacro (robot description, xacro)
@@ -5,4 +5,5 @@
     <xacro:include filename="$(find robot_description)/urdf/robot_gazebo.xacro"/>
     <!-- Link part_1 -->
+    <link name="base_footprint"/>
     <link name="base_link">
         <inertial>
@@ -52,8 +53,13 @@
         </collision>
     </link>
+    <joint name="base_joint" type="fixed">
+        <parent link="base_footprint"/>
+        <child link="base_link" />
+        <origin xyz="0 0 0" rpy="0 0 0"/>
+  </joint>
     <!-- Joint from part_1 to part_1_2 -->
     <joint name="right_wheel" type="continuous">
         <origin xyz="-0.480688 -0.0711889 0.605633" rpy="-1.5708 3.3994e-20 1.5708"/>
-        <parent link="part_1"/>
+        <parent link="base_link"/>
         <child link="part_1_2"/>
         <axis xyz="0 0 1"/>
@@ -88,5 +94,5 @@
     <joint name="left_wheel" type="continuous">
         <origin xyz="0.0616039 -0.0708403 0.609618" rpy="1.5708 -1.30234 1.5708"/>
-        <parent link="part_1"/>
+        <parent link="base_link"/>
         <child link="part_1_3"/>
         <axis xyz="0 0 1"/>

File: src/robot_description/urdf/robot.urdf.xacro (robot description, xacro)
@@ -5,4 +5,5 @@
     <xacro:include filename="$(find robot_description)/urdf/robot_gazebo.xacro"/>
     <!-- Link part_1 -->
+    <link name="base_footprint"/>
     <link name="base_link">
         <inertial>
@@ -52,4 +53,9 @@
         </collision>
     </link>
+    <joint name="base_joint" type="fixed">
+        <parent link="base_footprint"/>
+        <child link="base_link" />
+        <origin xyz="0 0 0" rpy="0 0 0"/>
+  </joint>
     <!-- Joint from part_1 to part_1_2 -->
     <joint name="right_wheel" type="continuous">
